File: scale/filament-scale-pcb.kicad_pcb (KiCad board)
At the start: 2 copper layers, 40.4 x 29.6 mm, 22 parts, among them J1 Load Cell, J2 MCU, J4 Peripherals, Q1 S9012, U1 HX711

Commit message: initial version for production
Parts:
- J4: footprint Connector_JST:JST_XH_B5B-XH-A_1x05_P2.50mm_Vertical -> Chof747_Connectors:JST_XH_B5B-XH-A_1x05_P2.54mm_Vertical
Changed lines of the file:
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@@
 		)
 	)
-	(footprint "Connector_JST:JST_XH_B5B-XH-A_1x05_P2.50mm_Vertical"
+	(footprint "Chof747_Connectors:JST_XH_B5B-XH-A_1x05_P2.54mm_Vertical"
 		(layer "F.Cu")
 		(at 146.8 55.3)
@@
 		(tags "connector JST XH vertical")
 		(property "Reference" "J4"
-			(at -3.6 0.5 0)
+			(at 5 -3.55 0)
 			(layer "F.SilkS")
 			(effects
@@
 		(property "Value" "Peripherals"
 			(at 5 4.6 0)
-			(layer "F.SilkS" knockout)
+			(layer "F.Fab")
 			(effects
 				(font
@@
 		(attr through_hole)
 		(fp_line
-			(start -2.85 -2.75)
-			(end -2.85 -1.5)
-			(stroke
-				(width 0.12)
-				(type solid)
-			)
-			(layer "F.SilkS")
-		)
-		(fp_line
-			(start -2.56 -2.46)
-			(end -2.56 3.51)
+			(start -2.93 -2.75)
+			(end -2.93 -1.5)
+			(stroke
+				(width 0.12)
+				(type solid)
+			)
+			(layer "F.SilkS")
+		)
+		(fp_line
+			(start -2.64 -2.46)
+			(end -2.64 3.51)
+			(stroke
+				(width 0.12)
+				(type solid)
+			)
+			(layer "F.SilkS")
+		)
+		(fp_line
+			(start -2.63 -2.45)
+			(end -2.63 -1.7)
+			(stroke
+				(width 0.12)
+				(type solid)
+			)
+			(layer "F.SilkS")
+		)
+		(fp_line
+			(start -2.63 -1.7)
+			(end -0.83 -1.7)
+			(stroke
+				(width 0.12)
+				(type solid)
+			)
+			(layer "F.SilkS")
+		)
+		(fp_line
+			(start -2.63 -0.2)
+			(end -1.88 -0.2)
 			(stroke
 				(width 0.12)
@@
 		(fp_line
 			(start -2.56 3.51)
-			(end 12.56 3.51)
-			(stroke
-				(width 0.12)
-				(type solid)
-			)
-			(layer "F.SilkS")
-		)
-		(fp_line
-			(start -2.55 -2.45)
-			(end -2.55 -1.7)
-			(stroke
-				(width 0.12)
-				(type solid)
-			)
-			(layer "F.SilkS")
-		)
-		(fp_line
-			(start -2.55 -1.7)
-			(end -0.75 -1.7)
-			(stroke
-				(width 0.12)
-				(type solid)
-			)
-			(layer "F.SilkS")
-		)
-		(fp_line
-			(start -2.55 -0.2)
-			(end -1.8 -0.2)
-			(stroke
-				(width 0.12)
-				(type solid)
-			)
-			(layer "F.SilkS")
-		)
-		(fp_line
-			(start -1.8 -0.2)
-			(end -1.8 2.75)
+			(end 12.64 3.51)
+			(stroke
+				(width 0.12)
+				(type solid)
+			)
+			(layer "F.SilkS")
+		)
+		(fp_line
+			(start -1.88 -0.2)
+			(end -1.88 2.75)
 			(stroke
 				(width 0.12)
@@
 		)
 		(fp_line
-			(start -1.6 -2.75)
-			(end -2.85 -2.75)
-			(stroke
-				(width 0.12)
-				(type solid)
-			)
-			(layer "F.SilkS")
-		)
-		(fp_line
-			(start -0.75 -2.45)
-			(end -2.55 -2.45)
-			(stroke
-				(width 0.12)
-				(type solid)
-			)
-			(layer "F.SilkS")
-		)
-		(fp_line
-			(start -0.75 -1.7)
-			(end -0.75 -2.45)
+			(start -1.68 -2.75)
+			(end -2.93 -2.75)
+			(stroke
+				(width 0.12)
+				(type solid)
+			)
+			(layer "F.SilkS")
+		)
+		(fp_line
+			(start -0.83 -2.45)
+			(end -2.63 -2.45)
+			(stroke
+				(width 0.12)
+				(type solid)
+			)
+			(layer "F.SilkS")
+		)
+		(fp_line
+			(start -0.83 -1.7)
+			(end -0.83 -2.45)
 			(stroke
 				(width 0.12)
@@
 		)
 		(fp_line
-			(start 10.75 -2.45)
-			(end 10.75 -1.7)
-			(stroke
-				(width 0.12)
-				(type solid)
-			)
-			(layer "F.SilkS")
-		)
-		(fp_line
-			(start 10.75 -1.7)
-			(end 12.55 -1.7)
-			(stroke
-				(width 0.12)
-				(type solid)
-			)
-			(layer "F.SilkS")
-		)
-		(fp_line
-			(start 11.8 -0.2)
-			(end 11.8 2.75)
-			(stroke
-				(width 0.12)
-				(type solid)
-			)
-			(layer "F.SilkS")
-		)
-		(fp_line
-			(start 11.8 2.75)
+			(start 10.83 -2.45)
+			(end 10.83 -1.7)
+			(stroke
+				(width 0.12)
+				(type solid)
+			)
+			(layer "F.SilkS")
+		)
+		(fp_line
+			(start 10.83 -1.7)
+			(end 12.63 -1.7)
+			(stroke
+				(width 0.12)
+				(type solid)
+			)
+			(layer "F.SilkS")
+		)
+		(fp_line
+			(start 11.88 -0.2)
+			(end 11.88 2.75)
+			(stroke
+				(width 0.12)
+				(type solid)
+			)
+			(layer "F.SilkS")
+		)
+		(fp_line
+			(start 11.88 2.75)
 			(end 5 2.75)
 			(stroke
@@
 		)
 		(fp_line
-			(start 12.55 -2.45)
-			(end 10.75 -2.45)
-			(stroke
-				(width 0.12)
-				(type solid)
-			)
-			(layer "F.SilkS")
-		)
-		(fp_line
-			(start 12.55 -1.7)
-			(end 12.55 -2.45)
-			(stroke
-				(width 0.12)
-				(type solid)
-			)
-			(layer "F.SilkS")
-		)
-		(fp_line
-			(start 12.55 -0.2)
-			(end 11.8 -0.2)
-			(stroke
-				(width 0.12)
-				(type solid)
-			)
-			(layer "F.SilkS")
-		)
-		(fp_line
-			(start 12.56 -2.46)
-			(end -2.56 -2.46)
-			(stroke
-				(width 0.12)
-				(type solid)
-			)
-			(layer "F.SilkS")
-		)
-		(fp_line
-			(start 12.56 3.51)
-			(end 12.56 -2.46)
+			(start 12.63 -2.45)
+			(end 10.83 -2.45)
+			(stroke
+				(width 0.12)
+				(type solid)
+			)
+			(layer "F.SilkS")
+		)
+		(fp_line
+			(start 12.63 -1.7)
+			(end 12.63 -2.45)
+			(stroke
+				(width 0.12)
+				(type solid)
+			)
+			(layer "F.SilkS")
+		)
+		(fp_line
+			(start 12.63 -0.2)
+			(end 11.88 -0.2)
+			(stroke
+				(width 0.12)
+				(type solid)
+			)
+			(layer "F.SilkS")
+		)
+		(fp_line
+			(start 12.64 -2.46)
+			(end -2.64 -2.46)
+			(stroke
+				(width 0.12)
+				(type solid)
+			)
+			(layer "F.SilkS")
+		)
+		(fp_line
+			(start 12.64 3.51)
+			(end 12.64 -2.46)
 			(stroke
 				(width 0.12)
@@
 		)
 		(fp_line
-			(start -2.45 -2.35)
-			(end -2.45 3.4)
+			(start -0.705 -2.35)
+			(end -0.08 -1.35)
 			(stroke
 				(width 0.1)
@@
 		)
 		(fp_line
-			(start -2.45 3.4)
-			(end 12.45 3.4)
-			(stroke
-				(width 0.1)
-				(type solid)
-			)
-			(layer "F.Fab")
-		)
-		(fp_line
-			(start -0.625 -2.35)
-			(end 0 -1.35)
-			(stroke
-				(width 0.1)
-				(type solid)
-			)
-			(layer "F.Fab")
-		)
-		(fp_line
-			(start 0 -1.35)
-			(end 0.625 -2.35)
-			(stroke
-				(width 0.1)
-				(type solid)
-			)
-			(layer "F.Fab")
-		)
-		(fp_line
-			(start 12.45 -2.35)
-			(end -2.45 -2.35)
-			(stroke
-				(width 0.1)
-				(type solid)
-			)
-			(layer "F.Fab")
-		)
-		(fp_line
-			(start 12.45 3.4)
-			(end 12.45 -2.35)
+			(start -0.08 -1.35)
+			(end 0.545 -2.35)
 			(stroke
 				(width 0.1)
@@
 		)
 		(pad "1" thru_hole roundrect
-			(at 0 0)
+			(at -0.08 0)
 			(size 1.7 1.95)
 			(drill 0.95)
@@
 		)
 		(pad "2" thru_hole oval
-			(at 2.5 0)
+			(at 2.46 0)
 			(size 1.7 1.95)
 			(drill 0.95)
@@
 		)
 		(pad "4" thru_hole oval
-			(at 7.5 0)
+			(at 7.54 0)
 			(size 1.7 1.95)
 			(drill 0.95)
@@
 		)
 		(pad "5" thru_hole oval
-			(at 10 0)
+			(at 10.08 0)
 			(size 1.7 1.95)
 			(drill 0.95)
@@
 		(polygon
 			(pts
-				(xy 121.3 72.3) (xy 130.5 72.3) (xy 130.5 77.4) (xy 140.4 77.4) (xy 140.4 69.7) (xy 144.1 69.7)
+				(xy 121.3 72.2) (xy 130.5 72.2) (xy 130.5 77.4) (xy 140.4 77.4) (xy 140.4 69.7) (xy 144.1 69.7)
 				(xy 144.196212 57) (xy 150.5 57) (xy 153.1 57) (xy 162.5 57) (xy 162.5 82.2) (xy 121.3 82.1)
 			)
