File: scale/filament-scale-pcb.kicad_sch (KiCad schematic)
At the start: 21 parts, among them J1 Load Cell, J2 MCU, J4 Peripherals, Q1 S9012, U1 HX711

Commit message: initial version for production
Parts:
- J4: footprint Connector_JST:JST_XH_B5B-XH-A_1x05_P2.50mm_Vertical -> Chof747_Connectors:JST_XH_B5B-XH-A_1x05_P2.54mm_Vertical
Changed lines of the file:
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@@
 			)
 		)
-		(property "Footprint" "Connector_JST:JST_XH_B5B-XH-A_1x05_P2.50mm_Vertical"
+		(property "Footprint" "Chof747_Connectors:JST_XH_B5B-XH-A_1x05_P2.54mm_Vertical"
 			(at 248.92 114.3 0)
 			(effects
