File: mcu-breakout/mcu-breakout.kicad_sch (KiCad schematic)
At the start: 20 parts, among them J1 SCALE 3, J2 SCALE 2, J3 SCALE 1, J4 Spare, J5 Environment, SW1 Mod, SW2 Reset

Commit message: changed to pico as a mcu
Parts:
- removed A1: Arduino_Nano_v3.x, Module:Arduino_Nano, symbol MCU_Module:Arduino_Nano_Every
- removed SW2: Reset, Chof747_Footprints:KEY-SMD_L3.9-W3.0-LS5.0-EH, symbol Switch:SW_Push
- added TP7: Clk 2, TestPoint:TestPoint_Pad_D2.0mm, symbol Connector:TestPoint
- added TP8: Clk 1, TestPoint:TestPoint_Pad_D2.0mm, symbol Connector:TestPoint
- added U1: RP2040-ZERO, Chof747_MCUs:RP2040-ZERO-THP, symbol Chof747_MCUs:RP2040-ZERO
- TP4: value Clk -> Clk 3
Connections:
- net +3V3 is gone; now on net SDA: J4.2 (Pin_2)
- net BTN_1: now also U1.10 (GP9)
- net BTN_2: now also U1.12 (GP11)
- net BTN_3: now also U1.14 (GP13)
- net BTN_MOD: now also U1.5 (GP4)
- net CLK_1: now also TP8.1, U1.20 (GP29)
- net CLK_2: now also TP7.1, U1.18 (GP27)
- net CLK_3: now also U1.16 (GP15)
- net DAT_1: now also U1.19 (GP28)
- net DAT_2: now also U1.17 (GP26)
- net DAT_3: now also U1.15 (GP14)
- net GND: now also U1.22 (GND)
- net LED_1: now also U1.9 (GP8)
- net LED_2: now also U1.11 (GP10)
- net LED_3: now also U1.13 (GP12)
- net SCL: now also J4.3 (Pin_3), U1.4 (GP3); no longer J4.4 (Pin_4)
- net SDA: now also U1.3 (GP2); no longer J4.3 (Pin_3)
- net VCC: now also U1.21 (3V3)
- net A6 renamed GP6
- net GP6: now also U1.7 (GP6)
- net A7 renamed GP7
- net GP7: now also U1.8 (GP7)
- net AREF renamed +5V
- net +5V: now also U1.23 (5V)
- new net GP5: J4.4 (Pin_4), U1.6 (GP5)
- no-connect marks 7 -> 2
