File: mcu-breakout/mcu-breakout.kicad_sch (KiCad schematic)
At the start: 20 parts, among them J1 SCALE 3, J2 SCALE 2, J3 SCALE 1, J4 Spare, J5 Environment, SW1 Mod, SW2 Reset

Commit message: initial version for production
Parts:
- J5: footprint Connector_JST:JST_XH_B4B-XH-A_1x04_P2.50mm_Vertical -> Chof747_Connectors:JST_XH_B4B-XH-A_1x04_P2.54mm_Vertical
Changed lines of the file:
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@@
 			)
 		)
-		(property "Footprint" "Connector_JST:JST_XH_B4B-XH-A_1x04_P2.50mm_Vertical"
+		(property "Footprint" "Chof747_Connectors:JST_XH_B4B-XH-A_1x04_P2.54mm_Vertical"
 			(at 104.14 147.32 0)
 			(effects

Commit message: Changed to separeted clock lines for the different scales
Connections:
- net SCL: now also J4.4 (Pin_4)
- net SDA: now also J4.3 (Pin_3)
- net A2 renamed CLK_1
- net CLK_1: now also J3.3 (Pin_3); no longer J4.3 (Pin_3)
- net A3 renamed CLK_2
- net CLK_2: now also J2.3 (Pin_3); no longer J4.4 (Pin_4)
- net CLK renamed CLK_3
- net CLK_3: no longer J2.3 (Pin_3), J3.3 (Pin_3)

Commit message: added schema print out and table with physical pin numbering to arduino version
Other:
- note added: "Bottom Right of Arduino Board Variant"
- note added: "Physical Pin Layout"
- note added: "Top Left of Arduino Board Variant"
- title: (none) -> Filament Scale MCU Breakout / Nano
